Commit message: pesan commit

File: robotta_description/urdf/gazebo_control.xacro (robot description, xacro)
@@ -6,6 +6,6 @@
             <left_joint>left_wheel_joint</left_joint>
             <right_joint>right_wheel_joint</right_joint>
-            <wheel_separation>0.35</wheel_separation>
-            <wheel_diameter>0.1</wheel_diameter>
+            <wheel_separation>0.5</wheel_separation>
+            <wheel_diameter>0.162</wheel_diameter>
             <!-- Limits -->
             <max_wheel_torque>200</max_wheel_torque>

File: robotta_description/urdf/robot_core.xacro (robot description, xacro)
@@ -5,5 +5,5 @@
     <xacro:property name="chassis_width" value="0.5"/>
     <xacro:property name="chassis_height" value="0.138"/>
-    <xacro:property name="chassis_mass" value="1.5"/>    <!-- nilai asal-->
+    <xacro:property name="chassis_mass" value="3.5"/>    <!-- nilai asal-->
     <xacro:property name="chassis_upper_length" value = "0.05"/>
     <xacro:property name="chassis_upper_width" value = "0.30"/>
@@ -11,5 +11,5 @@
     <xacro:property name="chassis_upper_mass" value = "0.01"/>
     <xacro:property name="chassis_offset_z" value = "${chassis_upper_height/2 + chassis_height/2}"/>
-    <xacro:property name="wheel_radius" value="0.0815"/>
+    <xacro:property name="wheel_radius" value="0.0825"/>
     <xacro:property name="wheel_thickness" value="0.05"/>
     <xacro:property name="wheel_mass" value="2.0"/>    <!-- nilai asal-->
@@ -18,5 +18,5 @@
     <xacro:property name="wheel_offset_z" value="0.05"/>
     <xacro:property name="caster_wheel_radius" value="0.03"/>
-    <xacro:property name="caster_wheel_mass" value="1.0"/>     <!-- nilai asal-->
+    <xacro:property name="caster_wheel_mass" value="1.5"/>     <!-- nilai asal-->
     <xacro:property name="caster_wheel_offset_x" value="0.45"/>
     <xacro:property name="caster_wheel_offset_y" value="0.20"/>  <!-- nilai asal-->

File: robotta_description/urdf/ros2_control.xacro (robot description, xacro)
@@ -5,5 +5,8 @@
             <hardware>
                 <plugin>robotta_hardware/RobottaHardware</plugin>
-                <param name="serial_port">/dev/ttyUSB1</param>
+                <param name="serial_port">/dev/ttyUSB0</param>
+                <!-- <param name="loop_rate">30</param>
+                <param name="timeout">1000</param>
+                <param name="enc_counts_per_rev">8999</param>  -->
             </hardware>
             <joint name="left_wheel_joint">

Commit message: adding new development

File: robotta_description/urdf/gazebo_control.xacro (robot description, xacro)
@@ -6,6 +6,6 @@
             <left_joint>left_wheel_joint</left_joint>
             <right_joint>right_wheel_joint</right_joint>
-            <wheel_separation>0.5</wheel_separation>
-            <wheel_diameter>0.162</wheel_diameter>
+            <wheel_separation>0.35</wheel_separation>
+            <wheel_diameter>0.1</wheel_diameter>
             <!-- Limits -->
             <max_wheel_torque>200</max_wheel_torque>

File: robotta_description/urdf/robot_core.xacro (robot description, xacro)
@@ -5,5 +5,5 @@
     <xacro:property name="chassis_width" value="0.5"/>
     <xacro:property name="chassis_height" value="0.138"/>
-    <xacro:property name="chassis_mass" value="3.5"/>    <!-- nilai asal-->
+    <xacro:property name="chassis_mass" value="1.5"/>    <!-- nilai asal-->
     <xacro:property name="chassis_upper_length" value = "0.05"/>
     <xacro:property name="chassis_upper_width" value = "0.30"/>
@@ -18,5 +18,5 @@
     <xacro:property name="wheel_offset_z" value="0.05"/>
     <xacro:property name="caster_wheel_radius" value="0.03"/>
-    <xacro:property name="caster_wheel_mass" value="1.5"/>     <!-- nilai asal-->
+    <xacro:property name="caster_wheel_mass" value="1.0"/>     <!-- nilai asal-->
     <xacro:property name="caster_wheel_offset_x" value="0.45"/>
     <xacro:property name="caster_wheel_offset_y" value="0.20"/>  <!-- nilai asal-->
@@ -25,4 +25,7 @@
         <color rgba="1 1 1 1" />
     </material>
+    <material name="gray">
+        <color rgba="0.6 0.6 0.6 1" />
+    </material>
     <material name="orange">
         <color rgba="1 0.3 0.1 1" />
@@ -60,5 +63,5 @@
                 <box size= "${chassis_length} ${chassis_width} ${chassis_height}" />   <!-- geometry dari rangka badan xyz = 30x30x15 cm-->
             </geometry>
-            <material name ="white"/>
+            <material name ="gray"/>
         </visual>
         <collision>
@@ -73,5 +76,5 @@
     </link>
     <gazebo reference="chassis">
-        <material>Gazebo/White</material>
+        <material>Gazebo/Gray</material>
     </gazebo>
     <!-- CHASSIS UPPER LINK -->
@@ -87,5 +90,5 @@
                 <box size= "${chassis_upper_length} ${chassis_upper_width} ${chassis_upper_height}" />   <!--geometry dari rangka badan xyz = 15x15x30 cm -->
             </geometry>
-            <material name ="white"/>
+            <material name ="gray"/>
         </visual>
         <collision>
@@ -101,5 +104,5 @@
     </link>
     <gazebo reference="chassis_upper">
-        <material>Gazebo/White</material>
+        <material>Gazebo/Gray</material>
     </gazebo>
     <!-- LEFT WHEEL LINK -->

File: robotta_description/urdf/ros2_control.xacro (robot description, xacro)
@@ -6,7 +6,4 @@
                 <plugin>robotta_hardware/RobottaHardware</plugin>
                 <param name="serial_port">/dev/ttyUSB0</param>
-                <!-- <param name="loop_rate">30</param>
-                <param name="timeout">1000</param>
-                <param name="enc_counts_per_rev">8999</param>  -->
             </hardware>
             <joint name="left_wheel_joint">
